Commit message: Update Gazebo and mobile base XACRO files

File: delivery_description/urdf/delivery_gazebo.xacro (robot description, xacro)
@@ -188,3 +188,103 @@
         </sensor>
     </gazebo>
+<!-- Ultrasonic Front Sensor -->
+<gazebo reference="ultrasonic_front_link">
+  <sensor name="ultrasonic_front" type="ray">
+    <always_on>true</always_on>
+    <update_rate>10</update_rate>
+    <visualize>true</visualize>
+    <topic>/ultrasonic/front</topic>
+    <gz_frame_id>ultrasonic_front_link</gz_frame_id>
+    <ray>
+      <scan>
+        <horizontal>
+          <samples>5</samples>
+          <resolution>1</resolution>
+          <min_angle>-0.05</min_angle>
+          <max_angle>0.05</max_angle>
+        </horizontal>
+      </scan>
+      <range>
+        <min>0.02</min>
+        <max>4.0</max>
+        <resolution>0.01</resolution>
+      </range>
+    </ray>
+  </sensor>
+</gazebo>
+<!-- Ultrasonic Back Sensor -->
+<gazebo reference="ultrasonic_back_link">
+  <sensor name="ultrasonic_back" type="ray">
+    <always_on>true</always_on>
+    <update_rate>10</update_rate>
+    <visualize>true</visualize>
+    <topic>/ultrasonic/back</topic>
+    <gz_frame_id>ultrasonic_back_link</gz_frame_id>
+    <ray>
+      <scan>
+        <horizontal>
+          <samples>5</samples>
+          <resolution>1</resolution>
+          <min_angle>-0.05</min_angle>
+          <max_angle>0.05</max_angle>
+        </horizontal>
+      </scan>
+      <range>
+        <min>0.02</min>
+        <max>4.0</max>
+        <resolution>0.01</resolution>
+      </range>
+    </ray>
+  </sensor>
+</gazebo>
+<!-- Ultrasonic Left Sensor -->
+<gazebo reference="ultrasonic_left_link">
+  <sensor name="ultrasonic_left" type="ray">
+    <always_on>true</always_on>
+    <update_rate>10</update_rate>
+    <visualize>true</visualize>
+    <topic>/ultrasonic/left</topic>
+    <gz_frame_id>ultrasonic_left_link</gz_frame_id>
+    <ray>
+      <scan>
+        <horizontal>
+          <samples>5</samples>
+          <resolution>1</resolution>
+          <min_angle>-0.05</min_angle>
+          <max_angle>0.05</max_angle>
+        </horizontal>
+      </scan>
+      <range>
+        <min>0.02</min>
+        <max>4.0</max>
+        <resolution>0.01</resolution>
+      </range>
+    </ray>
+  </sensor>
+</gazebo>
+<!-- Ultrasonic Right Sensor -->
+<gazebo reference="ultrasonic_right_link">
+  <sensor name="ultrasonic_right" type="ray">
+    <always_on>true</always_on>
+    <update_rate>10</update_rate>
+    <visualize>true</visualize>
+    <topic>/ultrasonic/right</topic>
+    <gz_frame_id>ultrasonic_right_link</gz_frame_id>
+    <ray>
+      <scan>
+        <horizontal>
+          <samples>5</samples>
+          <resolution>1</resolution>
+          <min_angle>-0.05</min_angle>
+          <max_angle>0.05</max_angle>
+        </horizontal>
+      </scan>
+      <range>
+        <min>0.02</min>
+        <max>4.0</max>
+        <resolution>0.01</resolution>
+      </range>
+    </ray>
+  </sensor>
+</gazebo>
 </robot>

File: delivery_description/urdf/delivery_mobile_base.xacro (robot description, xacro)
@@ -346,4 +346,57 @@
         <child link="camera_link_optical"/>
   </joint>
+  <!-- Ultrasonic Sensors -->
+<link name="ultrasonic_front_link">
+  <visual>
+    <geometry>
+      <cylinder radius="0.01" length="0.02"/>
+    </geometry>
+    <material name="blue"/>
+  </visual>
+</link>
+<joint name="ultrasonic_front_joint" type="fixed">
+  <parent link="base_link"/>
+  <child link="ultrasonic_front_link"/>
+  <origin xyz="0.28 0 0.08" rpy="0 0 0"/>
+</joint>
+<link name="ultrasonic_back_link">
+  <visual>
+    <geometry>
+      <cylinder radius="0.01" length="0.02"/>
+    </geometry>
+    <material name="blue"/>
+  </visual>
+</link>
+<joint name="ultrasonic_back_joint" type="fixed">
+  <parent link="base_link"/>
+  <child link="ultrasonic_back_link"/>
+  <origin xyz="-0.28 0 0.08" rpy="0 3.1416 0"/>
+</joint>
+<link name="ultrasonic_left_link">
+  <visual>
+    <geometry>
+      <cylinder radius="0.01" length="0.02"/>
+    </geometry>
+    <material name="blue"/>
+  </visual>
+</link>
+<joint name="ultrasonic_left_joint" type="fixed">
+  <parent link="base_link"/>
+  <child link="ultrasonic_left_link"/>
+  <origin xyz="0 0.28 0.08" rpy="0 0 1.5708"/>
+</joint>
+<link name="ultrasonic_right_link">
+  <visual>
+    <geometry>
+      <cylinder radius="0.01" length="0.02"/>
+    </geometry>
+    <material name="blue"/>
+  </visual>
+</link>
+<joint name="ultrasonic_right_joint" type="fixed">
+  <parent link="base_link"/>
+  <child link="ultrasonic_right_link"/>
+  <origin xyz="0 -0.28 0.08" rpy="0 0 -1.5708"/>
+</joint>
   <material name="blue">
     <color rgba="0 0 1 1"/>
